Commit message: fire_controller支持动态配置参数 删除rm_control包中的射速匹配曲线,移到friction_controller中实现 gimbal_controller关闭时会自动切断电机输出 修复test_usb_rc_py 修复了遥控器数据解析错误时不能丢包的bug 支持遥控器帧率统计 修改了部分电机ID 修改部分命名 修复了urdf错误配置导致pitch轴电机运行角度太小问题 rm_control支持角度限位 修复gimbal_controller中关于限位的逻辑错误的问题

File: robot_description_infantry/urdf/robot.urdf.xacro (robot description, xacro)
@@ -2,5 +2,5 @@
 <robot xmlns:xacro="http://www.ros.org/wiki/xacro" name="infantry-robot">
     <!-- Add transmission to urdf exported by Solidworks. -->
-    <xacro:macro name="motor_transmission" params="joint_name motor_name transmission_name motor_type">
+    <xacro:macro name="motor_transmission" params="joint_name motor_name transmission_name motor_type use_rotor">
         <transmission name="${transmission_name}">
             <type>transmission_interface/SimpleTransmission</type>
@@ -10,16 +10,21 @@
             </joint>
             <actuator name="${motor_name}">
-                <xacro:if value="${motor_type == 'RM3508'}">
-                    <mechanicalReduction>19</mechanicalReduction>
-                </xacro:if>
-                <xacro:if value="${motor_type == 'RM2006'}">
-                    <mechanicalReduction>36</mechanicalReduction>
-                </xacro:if>
-                <xacro:if value="${motor_type == 'RM6020'}">
+                <xacro:if value="${use_rotor}">
                     <mechanicalReduction>1</mechanicalReduction>
                 </xacro:if>
-                <xacro:if value="${motor_type == 'PWM'}">
-                    <mechanicalReduction>1</mechanicalReduction>
-                </xacro:if>
+                <xacro:unless value="${use_rotor}">
+                    <xacro:if value="${motor_type == 'RM3508'}">
+                        <mechanicalReduction>19</mechanicalReduction>
+                    </xacro:if>
+                    <xacro:if value="${motor_type == 'RM2006'}">
+                        <mechanicalReduction>36</mechanicalReduction>
+                    </xacro:if>
+                    <xacro:if value="${motor_type == 'RM6020'}">
+                        <mechanicalReduction>1</mechanicalReduction>
+                    </xacro:if>
+                    <xacro:if value="${motor_type == 'PWM'}">
+                        <mechanicalReduction>1</mechanicalReduction>
+                    </xacro:if>
+                </xacro:unless>
             </actuator>
         </transmission>
@@ -34,31 +39,31 @@
         <cylinder radius="0.07625" length="0.5"/>
     </xacro:macro>
-    <xacro:motor_transmission joint_name="base_to_left_forward_wheel_link"  motor_name="left_forward_motor"  transmission_name="left_forward_wheel_transmission"  motor_type="RM3508"/>
+    <xacro:motor_transmission joint_name="base_to_left_forward_wheel_link"  motor_name="left_forward_motor"  transmission_name="left_forward_wheel_transmission"  motor_type="RM3508" use_rotor="false"/>
     <xacro:macro name="collision_right_forward_wheel_link">
         <cylinder radius="0.07625" length="0.5"/>
     </xacro:macro>
-    <xacro:motor_transmission joint_name="base_to_right_forward_wheel_link" motor_name="right_forward_motor" transmission_name="right_forward_wheel_transmission" motor_type="RM3508"/>
+    <xacro:motor_transmission joint_name="base_to_right_forward_wheel_link" motor_name="right_forward_motor" transmission_name="right_forward_wheel_transmission" motor_type="RM3508" use_rotor="false"/>
     <xacro:macro name="collision_left_backward_wheel_link">
         <cylinder radius="0.07625" length="0.5"/>
     </xacro:macro>
-    <xacro:motor_transmission joint_name="base_to_left_backward_wheel_link"  motor_name="left_backward_motor"  transmission_name="left_backward_wheel_transmission"  motor_type="RM3508"/>
+    <xacro:motor_transmission joint_name="base_to_left_backward_wheel_link"  motor_name="left_backward_motor"  transmission_name="left_backward_wheel_transmission"  motor_type="RM3508" use_rotor="false"/>
     <xacro:macro name="collision_right_backward_wheel_link">
         <cylinder radius="0.07625" length="0.5"/>
     </xacro:macro>
-    <xacro:motor_transmission joint_name="base_to_right_backward_wheel_link" motor_name="right_backward_motor" transmission_name="right_backward_wheel_transmission" motor_type="RM3508"/>
+    <xacro:motor_transmission joint_name="base_to_right_backward_wheel_link" motor_name="right_backward_motor" transmission_name="right_backward_wheel_transmission" motor_type="RM3508" use_rotor="false"/>
     <!-- Gimbal -->
     <xacro:macro name="collision_yaw_link">
         <cylinder radius="0" length="0"/>
     </xacro:macro>
-    <xacro:motor_transmission joint_name="base_to_yaw_link"  motor_name="yaw_motor"  transmission_name="yaw_transmission"  motor_type="RM6020"/>
+    <xacro:motor_transmission joint_name="base_to_yaw_link"  motor_name="yaw_motor"  transmission_name="yaw_transmission"  motor_type="RM6020" use_rotor="true"/>
     <xacro:macro name="collision_pitch_link">
         <cylinder radius="0" length="0"/>
     </xacro:macro>
-    <xacro:motor_transmission joint_name="yaw_to_pitch_link"  motor_name="pitch_motor"  transmission_name="pitch_transmission"  motor_type="RM6020"/>
+    <xacro:motor_transmission joint_name="yaw_to_pitch_link"  motor_name="pitch_motor"  transmission_name="pitch_transmission"  motor_type="RM6020" use_rotor="true"/>
     <!-- Fire -->
     <xacro:macro name="collision_fire_link">
         <cylinder radius="0" length="0"/>
     </xacro:macro>
-    <xacro:motor_transmission joint_name="base_to_fire_link"  motor_name="fire_motor"  transmission_name="fire_transmission"  motor_type="RM2006"/>
+    <xacro:motor_transmission joint_name="base_to_fire_link"  motor_name="fire_motor"  transmission_name="fire_transmission"  motor_type="RM2006" use_rotor="false"/>
     <!-- Friction -->
     <link name="friction1_link"></link>
@@ -70,5 +75,5 @@
         <safety_controller k_position="9999" k_velocity="9999" soft_lower_limit="0" soft_upper_limit="0"/>
     </joint>
-    <xacro:motor_transmission joint_name="pitch_to_friction1_link"  motor_name="friction1_motor"  transmission_name="friction1_transmission"  motor_type="PWM"/>
+    <xacro:motor_transmission joint_name="pitch_to_friction1_link"  motor_name="friction1_motor"  transmission_name="friction1_transmission"  motor_type="RM2006" use_rotor="true"/>
     <link name="friction2_link"></link>
     <joint name="pitch_to_friction2_link" type="continuous">
@@ -79,5 +84,14 @@
         <safety_controller k_position="9999" k_velocity="9999" soft_lower_limit="0" soft_upper_limit="0"/>
     </joint>
-    <xacro:motor_transmission joint_name="pitch_to_friction2_link"  motor_name="friction2_motor"  transmission_name="friction2_transmission"  motor_type="PWM"/>
+    <xacro:motor_transmission joint_name="pitch_to_friction2_link"  motor_name="friction2_motor"  transmission_name="friction2_transmission"  motor_type="RM2006" use_rotor="true"/>
+    <link name="friction3_link"></link>
+    <joint name="pitch_to_friction3_link" type="continuous">
+        <parent link="pitch_link" />
+        <child link="friction3_link" />
+        <origin xyz="0 0 0" rpy="0 0 0" />
+        <limit effort="500" velocity="9999"/>
+        <safety_controller k_position="9999" k_velocity="9999" soft_lower_limit="0" soft_upper_limit="0"/>
+    </joint>
+    <xacro:motor_transmission joint_name="pitch_to_friction3_link"  motor_name="friction3_motor"  transmission_name="friction3_transmission"  motor_type="RM2006" use_rotor="true"/>
     <!-- Add dummy_link to prevent KDL error. -->
     <link name="dummy_link"></link>

Commit message: rm_control增加了射击控制 rm_control增加了射频限制 修改了部分注释和命名 裁判系统控制器支持删除UI话题 增加了对CKYF2305和Servo和PWM电机的支持 修复了一个巨大的map遍历写法导致程序崩溃的隐患 修复了ui框架对直线和矩形嵌套绘图时逻辑错误的问题 修复了鼠标按下时遥控器数据错误的问题 增加了UI对pitch角的显示 增加了UI调节准星功能 修改了sensor_imu包使其兼容python3 修复了电机指令发送错误的bug 修复了fire_controller读取参数错误问题 自定义UI增加小陀螺和弹舱盖状态显示

File: robot_description_infantry/urdf/robot.urdf.xacro (robot description, xacro)
@@ -7,5 +7,22 @@
             <joint name="${joint_name}">
                 <hardwareInterface>hardware_interface/JointStateInterface</hardwareInterface>
-                <hardwareInterface>hardware_interface/EffortJointInterface</hardwareInterface>
+                <xacro:if value="${motor_type == 'RM3508'}">
+                    <hardwareInterface>hardware_interface/EffortJointInterface</hardwareInterface>
+                </xacro:if>
+                <xacro:if value="${motor_type == 'RM2006'}">
+                    <hardwareInterface>hardware_interface/EffortJointInterface</hardwareInterface>
+                </xacro:if>
+                <xacro:if value="${motor_type == 'RM6020'}">
+                    <hardwareInterface>hardware_interface/EffortJointInterface</hardwareInterface>
+                </xacro:if>
+                <xacro:if value="${motor_type == 'PWM'}">
+                    <hardwareInterface>hardware_interface/VelocityJointInterface</hardwareInterface>
+                </xacro:if>
+                <xacro:if value="${motor_type == 'SERVO'}">
+                    <hardwareInterface>hardware_interface/PositionJointInterface</hardwareInterface>
+                </xacro:if>
+                <xacro:if value="${motor_type == 'CKYF2305'}">
+                    <hardwareInterface>hardware_interface/VelocityJointInterface</hardwareInterface>
+                </xacro:if>
             </joint>
             <actuator name="${motor_name}">
@@ -24,4 +41,10 @@
                     </xacro:if>
                     <xacro:if value="${motor_type == 'PWM'}">
+                        <mechanicalReduction>1</mechanicalReduction>
+                    </xacro:if>
+                    <xacro:if value="${motor_type == 'SERVO'}">
+                        <mechanicalReduction>1</mechanicalReduction>
+                    </xacro:if>
+                    <xacro:if value="${motor_type == 'CKYF2305'}">
                         <mechanicalReduction>1</mechanicalReduction>
                     </xacro:if>
@@ -94,4 +117,14 @@
     </joint>
     <xacro:motor_transmission joint_name="pitch_to_friction3_link"  motor_name="friction3_motor"  transmission_name="friction3_transmission"  motor_type="RM2006" use_rotor="true"/>
+    <!-- Bullet Cover -->
+    <link name="bullet_cover_link"></link>
+    <joint name="pitch_to_bullet_cover_link" type="continuous">
+        <parent link="pitch_link" />
+        <child link="bullet_cover_link" />
+        <origin xyz="0 0 0" rpy="0 0 0" />
+        <limit effort="500" velocity="9999"/>
+        <safety_controller k_position="9999" k_velocity="9999" soft_lower_limit="0" soft_upper_limit="0"/>
+    </joint>
+    <xacro:motor_transmission joint_name="pitch_to_bullet_cover_link"  motor_name="bullet_cover_motor"  transmission_name="bullet_cover_transmission"  motor_type="SERVO" use_rotor="false"/>
     <!-- Add dummy_link to prevent KDL error. -->
     <link name="dummy_link"></link>

Commit message: 电容电量支持曲线匹配 修改了toolbox中匹配曲线的逻辑 修复了function_generator的使用 修复了底盘跟随云台速度方向错误的问题 修复了小陀螺模式底盘跟随云台模块错误启用导致小陀螺模式速度不稳定的问题 针对19步兵车辆进行匹配 增加了rm_uI对弹舱盖状态是否显示的设定

File: robot_description_infantry/urdf/robot.urdf.xacro (robot description, xacro)
@@ -108,23 +108,4 @@
     </joint>
     <xacro:motor_transmission joint_name="pitch_to_friction2_link"  motor_name="friction2_motor"  transmission_name="friction2_transmission"  motor_type="PWM" use_rotor="true"/>
-    <link name="friction3_link"></link>
-    <joint name="pitch_to_friction3_link" type="continuous">
-        <parent link="pitch_link" />
-        <child link="friction3_link" />
-        <origin xyz="0 0 0" rpy="0 0 0" />
-        <limit effort="500" velocity="9999"/>
-        <safety_controller k_position="9999" k_velocity="9999" soft_lower_limit="0" soft_upper_limit="0"/>
-    </joint>
-    <xacro:motor_transmission joint_name="pitch_to_friction3_link"  motor_name="friction3_motor"  transmission_name="friction3_transmission"  motor_type="PWM" use_rotor="true"/>
-    <!-- Bullet Cover -->
-    <link name="bullet_cover_link"></link>
-    <joint name="pitch_to_bullet_cover_link" type="continuous">
-        <parent link="pitch_link" />
-        <child link="bullet_cover_link" />
-        <origin xyz="0 0 0" rpy="0 0 0" />
-        <limit effort="500" velocity="9999"/>
-        <safety_controller k_position="9999" k_velocity="9999" soft_lower_limit="0" soft_upper_limit="0"/>
-    </joint>
-    <xacro:motor_transmission joint_name="pitch_to_bullet_cover_link"  motor_name="bullet_cover_motor"  transmission_name="bullet_cover_transmission"  motor_type="SERVO" use_rotor="false"/>
     <!-- Add dummy_link to prevent KDL error. -->
     <link name="dummy_link"></link>
