Commit message: 修复了urdf的limit中力矩单位不正确的问题 删除了部分不必要的代码

File: robot_urdf_infantry/urdf/robot_urdf_infantry.urdf (robot description, URDF)
Before this commit: robot robot_urdf_infantry, 8 links, 7 joints
Joints:
- joint base_to_fire_link: limit effort=1080000 velocity=9999 -> effort=360 velocity=9999
- joint base_to_left_backward_wheel_link: limit effort=311296 velocity=9999 -> effort=380 velocity=9999
- joint base_to_left_forward_wheel_link: limit effort=311296 velocity=9999 -> effort=380 velocity=9999
- joint base_to_right_backward_wheel_link: limit effort=311296 velocity=9999 -> effort=380 velocity=9999
- joint base_to_right_forward_wheel_link: limit effort=311296 velocity=9999 -> effort=380 velocity=9999
- joint base_to_yaw_link: limit effort=10000 velocity=9999 -> effort=30 velocity=9999
- joint yaw_to_pitch_link: limit lower=-1.05 upper=1.5708 effort=10000 velocity=9999 -> lower=-1.05 upper=1.5708 effort=30 velocity=9999
